File: Hardware/Qwiic/SparkFun_Air_Quality_ENS160.brd (EAGLE design)
At the start: 25.4 x 25.4 mm, 59 parts, among them J1 QWIIC_RIGHT_ANGLE, J2 QWIIC_RIGHT_ANGLE, U1 AP2127K-1.8V, U24 ENS-160

Commit message: Fixes changes to ENS160
* In a panic I swapped pins rather than change the names on the pins - this has been undone. As a result I went to a previous version of the board and fixed the minor problems previously fixed:
* Fixes general ground pour problems
* Fixes silk
* Adds ADR to top pin
* Rolls version back to v10
* Changes VDD decoupling cap to 10uF - not 0.1uF
Parts:
- removed U$26: (no value), top:#POCI#16020
- added U$27: (no value), bot:##CS##441016
- U$22: device bot:##CS##441016 -> top:##CS##16019
- U$23: device top:##CS##16019 -> top:#POCI#16020
- U$8: device bot:#PICO#441017 -> bot:#ADR#441018
- moved U$24 5.08 mm to (11.4, 4.19)
- moved U$23 2.62 mm to (16.5, 4.06)
- moved U$21 0.28 mm to (21.2, 18.0)
- moved U$8 0.25 mm to (16.5, 3.94)
- moved ADDR 0.13 mm to (12.7, 15.2)
- moved U$14 0.13 mm to (9.40, 15.2)
- moved U$15 0.13 mm to (16.0, 15.2)
- moved U$6 0.13 mm to (12.7, 13.7)
- flipped U$22 to the bottom, turned to 270 degrees
Connections:
- removed net PICO/ADDR: ADDR.2, J3.5, U24.P1
- removed net POCI/SDA: J1.3, J2.3, J3.3, R2.1, U24.P3
- new net PICO/SDA: J1.3, J2.3, J3.3, R2.1, U24.P1
- new net POCI/ADDR: ADDR.2, J3.5, U24.P3
Routing:
- net POCI/SDA: track 54.4 -> 0.00 mm, vias 2 -> 0
- net PICO/SDA: track 0.00 -> 46.4 mm, vias 0 -> 2
- net PICO/ADDR: track 23.9 -> 0.00 mm, vias 3 -> 0
- net POCI/ADDR: track 0.00 -> 23.6 mm, vias 0 -> 2
- net GND: vias 30 -> 31

Commit message: Changes all values to 10k, removes pull up on interrupt
Parts:
- removed R5: 100k, SparkFun-Resistors:0603
- R6, R7, R8: value 100k -> 10k
- moved R3 0.25 mm to (17.1, 17.1)
- moved U1 0.25 mm to (17.1, 12.7)
- moved C1 0.25 mm to (17.1, 15.6)
- moved C2 0.25 mm to (17.1, 9.91)
- moved R6 0.25 mm to (17.1, 8.38)
- moved U$15 0.25 mm to (16.0, 15.0)
- moved R7 0.13 mm to (8.26, 17.1)
- moved R8 0.13 mm to (8.26, 15.6)
- renumbered U24 to U2
Connections:
- net !INT!: no longer R5.1
- net 3.3V: no longer R5.2
Routing:
- net 3.3V: track 70.8 -> 68.6 mm
- net !CS!: track 18.1 -> 16.6 mm
- net !INT!: track 18.8 -> 17.4 mm
- net GND: vias 31 -> 33

Commit message: Changes enable pin pullup to 10k on the VREG
Parts:
- R3: value 100k -> 10k
Changed lines of the file:
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@@
 <attribute name="VALUE" x="17.145" y="10.668" size="0.6096" layer="27" font="vector" ratio="20" rot="R180" align="top-center"/>
 </element>
-<element name="R3" library="SparkFun-Resistors" package="0603" value="100k" x="17.145" y="17.145" smashed="yes">
+<element name="R3" library="SparkFun-Resistors" package="0603" value="10k" x="17.145" y="17.145" smashed="yes">
 <attribute name="NAME" x="17.145" y="17.907" size="0.6096" layer="25" font="vector" ratio="20" align="bottom-center"/>
-<attribute name="PROD_ID" value="RES-07828" x="17.145" y="17.145" size="1.778" layer="27" display="off"/>
-<attribute name="VALUE" x="17.145" y="16.383" size="0.6096" layer="27" font="vector" ratio="20" align="top-center"/>
+<attribute name="PROD_ID" value="RES-00824" x="17.145" y="17.145" size="1.778" layer="27" display="off"/>
+<attribute name="VALUE" value="10k" x="17.145" y="16.383" size="0.6096" layer="27" font="vector" ratio="20" align="top-center"/>
 </element>
 <element name="R6" library="SparkFun-Resistors" package="0603" value="10k" x="17.145" y="8.382" smashed="yes">
