File: Hardware/SparkFun_Air_Quality_ENS160.sch (EAGLE design)
At the start: 31 parts, among them J1 QWIIC_RIGHT_ANGLE, J2 QWIIC_RIGHT_ANGLE, U1 AP2127K-1.8V, U2 ENS-160

Commit message: Fixes address selection notes
Other:
- note added: "Leave at VDD or OPEN for SPI Operation."
- note added: "Undefined"
- note removed: "SPI"
Changed lines of the file:
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@@
 <text x="66.04" y="88.9" size="1.778" layer="97" font="vector" align="center">0x52</text>
 <text x="66.04" y="93.98" size="1.778" layer="97" font="vector" align="center">0x53 (Default)</text>
-<text x="66.04" y="83.82" size="1.778" layer="97" font="vector" align="center">SPI</text>
+<text x="66.04" y="83.82" size="1.778" layer="97" font="vector" align="center">Undefined</text>
 <wire x1="35.56" y1="99.06" x2="53.34" y2="99.06" width="0.1524" layer="97" style="dashdot"/>
 <wire x1="53.34" y1="99.06" x2="52.578" y2="99.822" width="0.1524" layer="97" style="dashdot"/>
@@
 <text x="55.88" y="78.74" size="1.778" layer="97" font="vector" align="center">7-bit Unshifted</text>
 <text x="129.54" y="172.72" size="1.778" layer="97" font="vector" align="center">Input Range: 2.6V - 6V</text>
+<text x="38.1" y="104.14" size="1.27" layer="97" font="vector">Leave at VDD or
+OPEN for SPI
+Operation.</text>
 </plain>
 <instances>
