File: Hardware/SparkFun_Air_Quality_ENS160.sch (EAGLE design)
At the start: 31 parts, among them J1 QWIIC_RIGHT_ANGLE, J2 QWIIC_RIGHT_ANGLE, U1 AP2127K-1.8V, U2 ENS-160

Commit message: Removes unused library - new sensor added so SparkFun library
Parts:
- U2: device ENS160:ENS-160 -> SparkFun-Sensors:ENS-160
Changed lines of the file:
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@@
 <part name="FD4" library="SparkFun-Aesthetics" deviceset="FIDUCIAL" device="1X2"/>
 <part name="LOGO4" library="SparkFun-Aesthetics" deviceset="QWIIC_LOGO" device="_4MM"/>
-<part name="U2" library="ENS160" deviceset="ENS-160" device=""/>
+<part name="U2" library="SparkFun-Sensors" deviceset="ENS-160" device=""/>
 <part name="U1" library="SparkFun-IC-Power" deviceset="V_REG_AP2127" device="K-1.8V" value="AP2127K-1.8V"/>
 <part name="C1" library="SparkFun-Capacitors" deviceset="1.0UF" device="-0603-16V-10%" value="1.0uF"/>
@@
 <wire x1="53.34" y1="91.44" x2="78.74" y2="91.44" width="0.1524" layer="97"/>
 <wire x1="53.34" y1="86.36" x2="78.74" y2="86.36" width="0.1524" layer="97"/>
-<text x="45.72" y="93.98" size="1.778" layer="97" font="vector" align="center">VDD</text>
+<text x="45.72" y="93.98" size="1.778" layer="97" font="vector" ratio="15" align="center">VDD</text>
 <text x="45.72" y="88.9" size="1.778" layer="97" font="vector" align="center">GND</text>
 <text x="45.72" y="83.82" size="1.778" layer="97" font="vector" align="center">OPEN</text>
 <text x="66.04" y="88.9" size="1.778" layer="97" font="vector" align="center">0x52</text>
-<text x="66.04" y="93.98" size="1.778" layer="97" font="vector" align="center">0x53 (Default)</text>
+<text x="66.04" y="93.98" size="1.778" layer="97" font="vector" ratio="15" align="center">0x53 (Default)</text>
 <text x="66.04" y="83.82" size="1.778" layer="97" font="vector" align="center">Undefined</text>
 <wire x1="35.56" y1="99.06" x2="53.34" y2="99.06" width="0.1524" layer="97" style="dashdot"/>
