File: Hardware/SparkFun_Air_Quality_ENS160.brd (EAGLE design)
At the start: 25.4 x 25.4 mm, 58 parts, among them J1 QWIIC_RIGHT_ANGLE, J2 QWIIC_RIGHT_ANGLE, U1 AP2127K-1.8V, U2 ENS-160

Commit message: Removes unused library - new sensor added so SparkFun library
Parts:
- U2: device ENS160:LGA-9 -> SparkFun-Sensors:LGA-9
Changed lines of the file:
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@@
 <element name="LOGO4" library="SparkFun-Aesthetics" package="QWIIC_4MM" value="QWIIC_LOGO_4MM" x="2.6162" y="17.3482" smashed="yes"/>
 <element name="U$21" library="top" package="PWR9" value="" x="21.209" y="18.034" smashed="yes" rot="R90"/>
-<element name="U2" library="ENS160" package="LGA-9" value="ENS-160" x="12.7" y="12.7" smashed="yes">
+<element name="U2" library="SparkFun-Sensors" package="LGA-9" value="ENS-160" x="12.7" y="12.7" smashed="yes">
 <attribute name="NAME" x="11.0744" y="14.4272" size="0.6096" layer="25" font="vector" ratio="20"/>
 <attribute name="PROD_ID" value="IC-17100" x="12.7" y="12.7" size="1.778" layer="27" display="off"/>
